Commit message: Update lidar joint rotation to 180 degrees
Hi @Juancams,

I was chatting with @rodperex and we both think that the TF for the laser should match the current LiDAR setup, which is mounted on the Kobuki’s ceiling (flipped).

Let me know if you agree with this approach or if you prefer, we could add a xacro argument to keep things more flexible.

File: kobuki_description/urdf/sensors/lidar.urdf.xacro (robot description, xacro)
@@ -18,5 +18,5 @@
       </link>
       <joint name="$(arg namespace)laser_joint" type="fixed">
-        <origin xyz="0.0 0.0 0.37" rpy="0 0 0" />
+        <origin xyz="0.0 0.0 0.37" rpy="3.1416 0 0" />
         <parent link="$(arg namespace)base_link"/>
         <child link="$(arg namespace)laser_link" />
