Commit message: added arguments to change lidar position

File: kobuki_description/urdf/kobuki.urdf.xacro (robot description, xacro)
@@ -7,4 +7,10 @@
 <robot name="kobuki" xmlns:xacro="http://ros.org/wiki/xacro" >
   <xacro:arg name="lidar" default="false" />
+  <xacro:arg name="lidar_position_x" default="0" />
+  <xacro:arg name="lidar_position_y" default="0" />
+  <xacro:arg name="lidar_position_z" default="0.37" />
+  <xacro:arg name="lidar_orientation_roll" default="0" />
+  <xacro:arg name="lidar_orientation_pitch" default="0" />
+  <xacro:arg name="lidar_orientation_yaw" default="0" />
   <xacro:arg name="camera" default="false" />
   <xacro:arg name="structure" default="false" />
@@ -46,5 +52,11 @@
   <xacro:if value="$(arg lidar)">
     <xacro:include filename="$(find kobuki_description)/urdf/sensors/lidar.urdf.xacro"/>
-    <xacro:sensor_lidar namespace="$(arg namespace)"/>
+    <xacro:sensor_lidar namespace="$(arg namespace)"
+                        x="$(arg lidar_position_x)"
+                        y="$(arg lidar_position_y)"
+                        z="$(arg lidar_position_z)"
+                        roll="$(arg lidar_orientation_roll)"
+                        pitch="$(arg lidar_orientation_pitch)"
+                        yaw="$(arg lidar_orientation_yaw)"/>
   </xacro:if>
   <xacro:if value="$(arg camera)">

File: kobuki_description/urdf/sensors/lidar.urdf.xacro (robot description, xacro)
@@ -1,5 +1,5 @@
 <?xml version="1.0"?>
 <robot name="sensor_lidar" xmlns:xacro="http://ros.org/wiki/xacro">
-  <xacro:macro name="sensor_lidar" params = "namespace">
+  <xacro:macro name="sensor_lidar" params = "namespace x:=0 y:=0 z:=0.37 roll:=0 pitch:=0 yaw:=0">
   <link name="$(arg namespace)laser_link">
       <visual>
@@ -18,5 +18,5 @@
       </link>
       <joint name="$(arg namespace)laser_joint" type="fixed">
-        <origin xyz="0.0 0.0 0.37" rpy="3.1416 0 0" />
+        <origin xyz="${x} ${y} ${z}" rpy="${roll} ${pitch} ${yaw}" />
         <parent link="$(arg namespace)base_link"/>
         <child link="$(arg namespace)laser_link" />
